File: kicad/waffe_elektronik/waffe_elektronik.kicad_sch (KiCad schematic)
At the start: 80 parts, among them J1 WS2812 HP-Streifen, J2 GX16 7-polig, J3 USB-C (Flashen + Laden), M1 Vibromotor Rückstoss, M2 Vibromotor Treffer, Q1 AO3400A, Q2 AO3400A, Q3 AO3400A, SW1 Taster, SW2 Taster, SW3 RESET, SW4 BOOT, U1 MT3608, U10 TSOP34838, U11 TSOP34838, U12 USBLC6-2SC6, U2 AMS1117-3.3, U3 MCP73831, U4 ESP32-S3-WROOM-1-N16R8, U5 74HCT125, U6 MAX98357A, U7 TSOP34838, U8 TSOP34838, U9 TSOP34838

Commit message: Platine: Befestigung, OLED/Drehgeber, TSOP 6 an der Waffe, ein Vibrationsmotor
- 2 x M2-Befestigungslöcher (ISO 7380), kupferfrei auf allen Lagen
- OLED (I2C, Qwiic, J4) und Drehdrück-Geber (J5) an JST-SH 4 im neuen Streifen
  oben rechts, Platine L-förmig 59,6 x 46 mm
- Zweite TSAL6100 entfällt, an ihrem Platz J6 (JST-SH 3) für TSOP 6 an der Waffe (GPIO16),
  Filter am Sensor
- Nur noch ein Vibrationsmotor (GPIO47), GPIO48 frei; I2S-Leitungen kürzer
- Firmware: Pins für OLED/Geber, TSOP 6 auf GPIO16, ein Motor mit Prioritäten
- Schaltplan, Fertigungsdaten, Renders, Doku und Skills aktualisiert
Parts:
- removed D2: SS14, Diode_SMD:D_SOD-123F, symbol Diode:SS14
- removed LED2: TSAL6100, Connector_JST:JST_SH_SM02B-SRSS-TB_1x02-1MP_P1.00mm_Horizontal, symbol Device:LED
- removed M2: Vibromotor Treffer, Connector_JST:JST_SH_SM02B-SRSS-TB_1x02-1MP_P1.00mm_Horizontal, symbol Motor:Motor_DC
- removed Q3: AO3400A, Package_TO_SOT_SMD:SOT-23, symbol Transistor_FET:AO3400A
- removed R13: 100, Resistor_SMD:R_0603_1608Metric, symbol Device:R
- removed R14: 100k, Resistor_SMD:R_0603_1608Metric, symbol Device:R
- removed R8: 10, Resistor_SMD:R_1206_3216Metric, symbol Device:R
- added C24: 4.7u, symbol Device:C_Polarized
- added J4: OLED I²C (Qwiic), Connector_JST:JST_SH_SM04B-SRSS-TB_1x04-1MP_P1.00mm_Horizontal, symbol Connector_Generic:Conn_01x04
- added J5: Drehgeber, Connector_JST:JST_SH_SM04B-SRSS-TB_1x04-1MP_P1.00mm_Horizontal, symbol Connector_Generic:Conn_01x04
- added J6: TSOP 6 (Waffe), Connector_JST:JST_SH_SM03B-SRSS-TB_1x03-1MP_P1.00mm_Horizontal, symbol Connector_Generic:Conn_01x03
- added R26: 100, symbol Device:R
- added U13: TSOP34838, symbol Interface_Optical:TSOP348xx
- M1: value Vibromotor Rückstoss -> Vibromotor
Connections:
- net 3V3_MCU: now also J4.2 (Pin_2), J6.1 (Pin_1), R26.1
- net GND: now also C24.2, J4.1 (Pin_1), J5.1 (Pin_1), J6.2 (Pin_2), U13.2 (GND)
- net ENC_SW: now reaches U4.17 (IO9)
- net ENC_SW: now also J5.2 (Pin_2)
- net ENC_B: now reaches U4.34 (IO41)
- net ENC_B: now also J5.3 (Pin_3)
- net ENC_A: now reaches U4.35 (IO42)
- net ENC_A: now also J5.4 (Pin_4)
- net I2C_SDA: now reaches U4.38 (IO2)
- net I2C_SDA: now also J4.3 (Pin_3)
- net I2C_SCL: now reaches U4.39 (IO1)
- net I2C_SCL: now also J4.4 (Pin_4)
- net TSOP6_OUT: now reaches U4.9 (IO16)
- net TSOP6_OUT: now also J6.3 (Pin_3), U13.1 (OUT)
- net HIT_VIB renamed VIB
- net VIB: now also R11.1
- net RECOIL_VIB: no longer names the net of U4.25 (IO48)
- net RECOIL_VIB: no longer R11.1
- new net: C24.1, R26.2, U13.3 (Vs)
- no-connect marks 22 -> 17
Other:
- note added: "Bedienung: OLED + Drehgeber"
- note added: "IR-Sender (TSAL6100)"
- note added: "Kabel zum Sensor an der Waffe"
- note added: "Pull-ups für I²C auf dem OLED-Modul, Drehgeber über interne Pull-ups"
- note added: "TSOP 6 (an der Waffe, jenseits des Steckers)"
- note added: "Vibration (Rückstoss + Treffer)"
- note added: "Waffe vorne"
- note added: "frei: IO7, IO15, IO21, IO48"
- note removed: "IO21 reserviert: TSOP 6 (Waffe vorne)"
- note removed: "IR-Sender (2× TSAL6100 parallel)"
- note removed: "Rückstoss- / Treffer-Vibration"
- note removed: "frei: IO1/IO2 (Munitions-LED / I²C), IO7, IO9, IO15/16, IO41/42"

Commit message: Platine: USB-C senkrecht (HRO TYPE-C-31-E-17), Stecker durch die Seitenwand
- J3 jetzt senkrechte, wasserdichte USB-C-Buchse (LCSC C7424785), eigener Footprint in
  footprints/lasertag.pretty (fp-lib-table), 3D-Modell per gen_3d_usb_c_vertical.py
- USB-Paar neu geroutet: D+ über Via in der Buchsenmitte, D- über B.Cu-Brücke mit Abgriff
  in der Mitte; beide Steckrichtungen gleich lang (<= 0,007 mm), je 2 Vias
- CC2-Widerstand R22 unter der Buchse, R23 daneben; VBUS-Ring auf B.Cu
- Schaltplan, Fertigungsdaten, Renders, Doku und Skill aktualisiert
Parts:
- J3: footprint Connector_USB:USB_C_Receptacle_GCT_USB4105-xx-A_16P_TopMnt_Horizontal -> lasertag:USB_C_Receptacle_HRO_TYPE-C-31-E-17_Vertical; LCSC C5184243 -> C7424785
Changed lines of the file:
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@@
       (effects (font (size 1.27 1.27)))
     )
-    (property "Footprint" "Connector_USB:USB_C_Receptacle_GCT_USB4105-xx-A_16P_TopMnt_Horizontal" (at 0 0 0)
+    (property "Footprint" "lasertag:USB_C_Receptacle_HRO_TYPE-C-31-E-17_Vertical" (at 0 0 0)
       (effects (font (size 1.27 1.27)) hide)
     )
-    (property "LCSC" "C5184243" (at 0 0 0)
+    (property "LCSC" "C7424785" (at 0 0 0)
       (effects (font (size 1.27 1.27)) hide)
     )
