File: kicad/waffe_elektronik/waffe_elektronik.kicad_sch (KiCad schematic)
At the start: 79 parts, among them J1 WS2812 HP-Streifen, J2 GX16 7-polig, J3 USB-C (Flashen + Laden), J4 OLED I²C (Qwiic), J5 Drehgeber, J6 TSOP 6 (Waffe), M1 Vibromotor, Q1 AO3400A, Q2 AO3400A, SW1 Taster, SW2 Taster, SW3 RESET, SW4 BOOT, U1 MT3608, U10 TSOP34838, U11 TSOP34838, U12 USBLC6-2SC6, U13 TSOP34838, U2 AMS1117-3.3, U3 MCP73831, U4 ESP32-S3-WROOM-1-N16R8, U5 74HCT125, U6 MAX98357A, U7 TSOP34838, U8 TSOP34838, U9 TSOP34838

Commit message: Platine: Stecker nach Kabelwegen ausgerichtet, USB-C bündig mit der Gehäusewand
J1/SP1 an die linke Kante (Hauptschacht), SW1/SW2 an die Unterkante (Kanal zum
Abzugsschalter), J2 rechts unter M1 (Motorschacht), RESET auf den EN-Weg.
USB-C hanxia HX-TYPE-C 16P 180 LT H10.5 (10,5 mm), neues USB-Routing, Paar gleich lang.
J1 auf CJT A2001WR-S-3P (Lager). Gehäuse: Zonen, USB-Durchbruch mit Mulde,
Nachladetaste 5 mm nach hinten. Kabelwege, Fertigungsdaten, Bilder, READMEs neu.
Parts:
- J1: LCSC C265101 -> C225234
- J3: footprint lasertag:USB_C_Receptacle_HRO_TYPE-C-31-E-17_Vertical -> lasertag:USB_C_Receptacle_HX_TYPE-C-16P-180-LT-H10.5_Vertical; LCSC C7424785 -> C49261570
Changed lines of the file:
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@@
       (effects (font (size 1.27 1.27)))
     )
-    (property "Footprint" "lasertag:USB_C_Receptacle_HRO_TYPE-C-31-E-17_Vertical" (at 0 0 0)
-      (effects (font (size 1.27 1.27)) hide)
-    )
-    (property "LCSC" "C7424785" (at 0 0 0)
+    (property "Footprint" "lasertag:USB_C_Receptacle_HX_TYPE-C-16P-180-LT-H10.5_Vertical" (at 0 0 0)
+      (effects (font (size 1.27 1.27)) hide)
+    )
+    (property "LCSC" "C49261570" (at 0 0 0)
       (effects (font (size 1.27 1.27)) hide)
     )
@@
       (effects (font (size 1.27 1.27)) (justify left) hide)
     )
-    (property "LCSC" "C265101" (at 0 0 0)
-      (effects (font (size 1.27 1.27)) (justify left) hide)
-    )
+    (property "LCSC" "C225234" (at 0 0 0)
+      (effects (font (size 1.27 1.27)) (justify left) hide)
+    )

Commit message: Platine: Flash 128 MB, microSD-Slot, Akkuschutz; Schaltplan auf fünf Seiten
- SPI-NAND GD5F1GQ5UEYIGR (U14, 128 MB) für Audio-Dateien an IO7/IO15/IO3/IO46
- microSD-Slot TF-018 (J7, Push-Pull) am selben SPI-Bus, /CS an IO48, DAT1/DAT2 mit Pull-up
- Akkuschutz DW01A + FS8205A in einer Lasche oben links neben BT1
- USB versorgt 5V_PERIPH über SS14 (Flashen ohne Akku), STAT über BAT54WS an IO18
- C7 als IR-Puffer an GND, TSOP-Leitungen über 100 Ω an J2
- Platine 59,6 × 51 mm, J2 an der rechten Kante, H2 versetzt, Gehäusetasche und Kabelwege angepasst
- Schaltplan hierarchisch: Übersicht + fünf A3-Seiten, Projekt-Symbolbibliothek, ERC ohne Meldungen
Parts:
- removed BT1: 1S LiPo 3,7 V, Connector_JST:JST_PH_S2B-PH-SM4-TB_1x02-1MP_P2.00mm_Horizontal, symbol Device:Battery_Cell
- removed C1, C10, C7: 100u, Capacitor_SMD:C_1210_3225Metric, symbol Device:C
- removed C11, C12, C13, C14, C15, C24: 4.7u, symbol Device:C_Polarized
- removed C16, C4, C5: 1u, Capacitor_SMD:C_0603_1608Metric, symbol Device:C
- removed C17, C21, C23, C6, C8, C9: 100n, Capacitor_SMD:C_0603_1608Metric, symbol Device:C
- removed C18, C2, C22: 10u, Capacitor_SMD:C_0805_2012Metric, symbol Device:C
- removed C19, C20: 22u, Capacitor_SMD:C_0805_2012Metric, symbol Device:C
- removed C3: 10u, Capacitor_Tantalum_SMD:CP_EIA-3528-21_Kemet-B, symbol Device:C_Polarized
- removed D1: SS14, Diode_SMD:D_SOD-123F, symbol Diode:SS14
- removed D3: SS34, Diode_SMD:D_SMA, symbol Diode:SS34
- removed J1: WS2812 HP-Streifen, Connector_JST:JST_PH_S3B-PH-SM4-TB_1x03-1MP_P2.00mm_Horizontal, symbol Connector_Generic:Conn_01x03
- removed J2: GX16 7-polig, Connector_JST:JST_SH_SM07B-SRSS-TB_1x07-1MP_P1.00mm_Horizontal, symbol Connector_Generic:Conn_01x07
- removed J3: USB-C (Flashen + Laden), lasertag:USB_C_Receptacle_HX_TYPE-C-16P-180-LT-H10.5_Vertical, symbol Connector:USB_C_Receptacle_USB2.0_16P
- removed J4: OLED I²C (Qwiic), Connector_JST:JST_SH_SM04B-SRSS-TB_1x04-1MP_P1.00mm_Horizontal, symbol Connector_Generic:Conn_01x04
- removed J5: Drehgeber, Connector_JST:JST_SH_SM04B-SRSS-TB_1x04-1MP_P1.00mm_Horizontal, symbol Connector_Generic:Conn_01x04
- removed J6: TSOP 6 (Waffe), Connector_JST:JST_SH_SM03B-SRSS-TB_1x03-1MP_P1.00mm_Horizontal, symbol Connector_Generic:Conn_01x03
- removed L1: 10u, Inductor_SMD:L_Sunlord_MWSA0503S, symbol Device:L
- removed LED1: TSAL6100, Connector_JST:JST_SH_SM02B-SRSS-TB_1x02-1MP_P1.00mm_Horizontal, symbol Device:LED
- removed M1: Vibromotor, Connector_JST:JST_SH_SM02B-SRSS-TB_1x02-1MP_P1.00mm_Horizontal, symbol Motor:Motor_DC
- removed Q1, Q2: AO3400A, Package_TO_SOT_SMD:SOT-23, symbol Transistor_FET:AO3400A
- removed R1: 2k, Resistor_SMD:R_0603_1608Metric, symbol Device:R
- removed R10, R2, R21, R25, R9: 10k, Resistor_SMD:R_0603_1608Metric, symbol Device:R
- removed R11, R5: 100, Resistor_SMD:R_0603_1608Metric, symbol Device:R
- removed R12, R3, R4, R6: 100k, Resistor_SMD:R_0603_1608Metric, symbol Device:R
- removed R15: 330, Resistor_SMD:R_0603_1608Metric, symbol Device:R
- removed R16, R17, R18, R19, R20, R26: 100, symbol Device:R
- removed R22, R23: 5.1k, Resistor_SMD:R_0603_1608Metric, symbol Device:R
- removed R24: 75k, Resistor_SMD:R_0603_1608Metric, symbol Device:R
- removed R7: 10, Resistor_SMD:R_1206_3216Metric, symbol Device:R
- removed SP1: Lautsprecher, Connector_JST:JST_PH_S2B-PH-SM4-TB_1x02-1MP_P2.00mm_Horizontal, symbol Device:Speaker
- removed SW1, SW2: Taster, Connector_JST:JST_SH_SM02B-SRSS-TB_1x02-1MP_P1.00mm_Horizontal, symbol Switch:SW_Push
- removed SW3: RESET, Button_Switch_SMD:SW_SPST_B3U-1000P, symbol Switch:SW_Push
- removed SW4: BOOT, Button_Switch_SMD:SW_SPST_B3U-1000P, symbol Switch:SW_Push
- removed U1: MT3608, Package_TO_SOT_SMD:SOT-23-6, symbol Regulator_Switching:MT3608
- removed U10, U11, U13, U7, U8, U9: TSOP34838, symbol Interface_Optical:TSOP348xx
- removed U12: USBLC6-2SC6, Package_TO_SOT_SMD:SOT-23-6, symbol Power_Protection:USBLC6-2SC6
- removed U2: AMS1117-3.3, Package_TO_SOT_SMD:SOT-223-3_TabPin2, symbol Regulator_Linear:AMS1117-3.3
- removed U3: MCP73831, Package_TO_SOT_SMD:SOT-23-5, symbol Battery_Management:MCP73831-2-OT
- removed U4: ESP32-S3-WROOM-1-N16R8, RF_Module:ESP32-S3-WROOM-1, symbol RF_Module:ESP32-S3-WROOM-1
- removed U5: 74HCT125, Package_SO:TSSOP-14_4.4x5mm_P0.65mm, symbol 74xx:74AHCT125
- removed U6: MAX98357A, Package_DFN_QFN:TQFN-16-1EP_3x3mm_P0.5mm_EP1.23x1.23mm, symbol Audio:MAX98357A
Connections:
- no-connect marks 17 -> 0
Other:
- added sheet Audio und Speicher (audio_speicher.kicad_sch)
- added sheet Bedienung und Aktoren (bedienung_aktoren.kicad_sch)
- added sheet ESP32-S3 und USB (mcu_usb.kicad_sch)
- added sheet Sensoren (sensoren.kicad_sch)
- added sheet Stromversorgung (stromversorgung.kicad_sch)
- note added: "Signale zwischen den Seiten über globale Labels, Versorgung über Power-Symbole"
- note removed: "Abzug / Nachladen"
- note removed: "Akku-Messung"
- note removed: "Bedienung: OLED + Drehgeber"
- note removed: "Brust"
- note removed: "ESP32-S3-WROOM-1"
- note removed: "IR-Sender (TSAL6100)"
- note removed: "Kabel zum Sensor an der Waffe"
- note removed: "Laden (USB-C)"
- note removed: "Pull-ups für I²C auf dem OLED-Modul, Drehgeber über interne Pull-ups"
- note removed: "Rücken"
- note removed: "Schultern"
- note removed: "Sensorkabel zur Weste"
- note removed: "Sound (I²S)"
- note removed: "Stirnband hinten"
- note removed: "Stirnband vorn"
- note removed: "Stromversorgung"
- note removed: "TSOP 6 (an der Waffe, jenseits des Steckers)"
- note removed: "USB-C (nativer USB des ESP32-S3)"
- note removed: "Vibration (Rückstoss + Treffer)"
- note removed: "WS2812 (5 V) über Pegelwandler"
- note removed: "Waffe vorne"
- note removed: "Weste (nur Sensoren, jenseits des Steckers)"
- note removed: "frei: IO7, IO15, IO21, IO48"
- note removed: "unbenutzte Gatter: Eingänge + /OE auf GND"
- title: Lasertag - Waffen-Elektronik -> Lasertag - Waffen-Elektronik: Übersicht
