File: kicad/waffe_elektronik/audio_speicher.kicad_sch (KiCad schematic)
At the start: 10 parts, among them J7 TF-018, U14 GD5F1GQ5UEYIGR, U6 MAX98357A

Commit message: Platine: günstigere JLC-Teile, Option ESP32-S3-WROOM-1U mit externer Antenne
- Flash ZD35Q1GC-IB, Kondensatoren/Dioden/Widerstände auf Basic-Teile und 0402, Layout angepasst
- WROOM-1U auf demselben Footprint: eigene JLCPCB-BOM/CPL (Modulmitte 3,15 mm versetzt),
  Mouser-Option mit Pigtail RP-SMA/U.FL und Knick-Stabantenne, 3D-Modell des 1U
- Gerber, BOM, CPL, Renders und Bestelllisten neu erzeugt

Co-Authored-By: Claude Opus 5.5 <noreply@anthropic.com>
Claude-Session: https://claude.ai/code/session_01KkZzubjLKyW9odUwvmxTog
Parts:
- SP1: LCSC C225233 -> (none)
- U14: value GD5F1GQ5UEYIGR -> ZD35Q1GC-IB; LCSC C2829047 -> C2928927
Changed lines of the file:
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@@
     (instances
       (project "waffe_elektronik"
-        (path "/01404002-de85-4f35-b413-98d5163e0060"
+        (path "/9749138d-5476-4991-b12a-e9f07c79da08"
           (reference "U6") (unit 1)
         )
@@
     (instances
       (project "waffe_elektronik"
-        (path "/01404002-de85-4f35-b413-98d5163e0060"
+        (path "/9749138d-5476-4991-b12a-e9f07c79da08"
           (reference "#PWR70") (unit 1)
         )
@@
     (instances
       (project "waffe_elektronik"
-        (path "/01404002-de85-4f35-b413-98d5163e0060"
+        (path "/9749138d-5476-4991-b12a-e9f07c79da08"
           (reference "C22") (unit 1)
         )
@@
     (instances
       (project "waffe_elektronik"
-        (path "/01404002-de85-4f35-b413-98d5163e0060"
+        (path "/9749138d-5476-4991-b12a-e9f07c79da08"
           (reference "#PWR71") (unit 1)
         )
@@
     (instances
       (project "waffe_elektronik"
-        (path "/01404002-de85-4f35-b413-98d5163e0060"
+        (path "/9749138d-5476-4991-b12a-e9f07c79da08"
           (reference "C23") (unit 1)
         )
@@
     (instances
       (project "waffe_elektronik"
-        (path "/01404002-de85-4f35-b413-98d5163e0060"
+        (path "/9749138d-5476-4991-b12a-e9f07c79da08"
           (reference "#PWR72") (unit 1)
         )
@@
     (instances
       (project "waffe_elektronik"
-        (path "/01404002-de85-4f35-b413-98d5163e0060"
+        (path "/9749138d-5476-4991-b12a-e9f07c79da08"
           (reference "#PWR73") (unit 1)
         )
@@
     (instances
       (project "waffe_elektronik"
-        (path "/01404002-de85-4f35-b413-98d5163e0060"
+        (path "/9749138d-5476-4991-b12a-e9f07c79da08"
           (reference "#PWR74") (unit 1)
         )
@@
     (instances
       (project "waffe_elektronik"
-        (path "/01404002-de85-4f35-b413-98d5163e0060"
+        (path "/9749138d-5476-4991-b12a-e9f07c79da08"
           (reference "#PWR75") (unit 1)
         )
@@
       (effects (font (size 1.27 1.27)) (justify left) hide)
     )
-    (property "LCSC" "C225233" (at 0 0 0)
-      (effects (font (size 1.27 1.27)) (justify left) hide)
-    )
-    (pin "1")
-    (pin "2")
-    (instances
-      (project "waffe_elektronik"
-        (path "/01404002-de85-4f35-b413-98d5163e0060"
+    (pin "1")
+    (pin "2")
+    (instances
+      (project "waffe_elektronik"
+        (path "/9749138d-5476-4991-b12a-e9f07c79da08"
           (reference "SP1") (unit 1)
         )
@@
       (effects (font (size 1.27 1.27)) (justify left))
     )
-    (property "Value" "GD5F1GQ5UEYIGR" (at 146.05 85.09 0)
+    (property "Value" "ZD35Q1GC-IB" (at 146.05 85.09 0)
       (effects (font (size 1.27 1.27)) (justify left))
     )
@@
       (effects (font (size 1.27 1.27)) (justify left) hide)
     )
-    (property "LCSC" "C2829047" (at 0 0 0)
+    (property "LCSC" "C2928927" (at 0 0 0)
       (effects (font (size 1.27 1.27)) (justify left) hide)
     )
@@
     (instances
       (project "waffe_elektronik"
-        (path "/01404002-de85-4f35-b413-98d5163e0060"
+        (path "/9749138d-5476-4991-b12a-e9f07c79da08"
           (reference "U14") (unit 1)
         )
@@
     (instances
       (project "waffe_elektronik"
-        (path "/01404002-de85-4f35-b413-98d5163e0060"
+        (path "/9749138d-5476-4991-b12a-e9f07c79da08"
           (reference "#PWR76") (unit 1)
         )
@@
     (instances
       (project "waffe_elektronik"
-        (path "/01404002-de85-4f35-b413-98d5163e0060"
+        (path "/9749138d-5476-4991-b12a-e9f07c79da08"
           (reference "C25") (unit 1)
         )
@@
     (instances
       (project "waffe_elektronik"
-        (path "/01404002-de85-4f35-b413-98d5163e0060"
+        (path "/9749138d-5476-4991-b12a-e9f07c79da08"
           (reference "#PWR77") (unit 1)
         )
@@
     (instances
       (project "waffe_elektronik"
-        (path "/01404002-de85-4f35-b413-98d5163e0060"
+        (path "/9749138d-5476-4991-b12a-e9f07c79da08"
           (reference "#PWR78") (unit 1)
         )
@@
     (instances
       (project "waffe_elektronik"
-        (path "/01404002-de85-4f35-b413-98d5163e0060"
+        (path "/9749138d-5476-4991-b12a-e9f07c79da08"
           (reference "R27") (unit 1)
         )
@@
     (instances
       (project "waffe_elektronik"
-        (path "/01404002-de85-4f35-b413-98d5163e0060"
+        (path "/9749138d-5476-4991-b12a-e9f07c79da08"
           (reference "#PWR79") (unit 1)
         )
@@
     (instances
       (project "waffe_elektronik"
-        (path "/01404002-de85-4f35-b413-98d5163e0060"
+        (path "/9749138d-5476-4991-b12a-e9f07c79da08"
           (reference "#PWR80") (unit 1)
         )
@@
     (instances
       (project "waffe_elektronik"
-        (path "/01404002-de85-4f35-b413-98d5163e0060"
+        (path "/9749138d-5476-4991-b12a-e9f07c79da08"
           (reference "J7") (unit 1)
         )
@@
     (instances
       (project "waffe_elektronik"
-        (path "/01404002-de85-4f35-b413-98d5163e0060"
+        (path "/9749138d-5476-4991-b12a-e9f07c79da08"
           (reference "R37") (unit 1)
         )
@@
     (instances
       (project "waffe_elektronik"
-        (path "/01404002-de85-4f35-b413-98d5163e0060"
+        (path "/9749138d-5476-4991-b12a-e9f07c79da08"
           (reference "#PWR81") (unit 1)
         )
@@
     (instances
       (project "waffe_elektronik"
-        (path "/01404002-de85-4f35-b413-98d5163e0060"
+        (path "/9749138d-5476-4991-b12a-e9f07c79da08"
           (reference "#PWR82") (unit 1)
         )
@@
     (instances
       (project "waffe_elektronik"
-        (path "/01404002-de85-4f35-b413-98d5163e0060"
+        (path "/9749138d-5476-4991-b12a-e9f07c79da08"
           (reference "#PWR83") (unit 1)
         )
@@
     (instances
       (project "waffe_elektronik"
-        (path "/01404002-de85-4f35-b413-98d5163e0060"
+        (path "/9749138d-5476-4991-b12a-e9f07c79da08"
           (reference "#PWR84") (unit 1)
         )
@@
     (instances
       (project "waffe_elektronik"
-        (path "/01404002-de85-4f35-b413-98d5163e0060"
+        (path "/9749138d-5476-4991-b12a-e9f07c79da08"
           (reference "C26") (unit 1)
         )
@@
     (instances
       (project "waffe_elektronik"
-        (path "/01404002-de85-4f35-b413-98d5163e0060"
+        (path "/9749138d-5476-4991-b12a-e9f07c79da08"
           (reference "#PWR85") (unit 1)
         )
@@
     (instances
       (project "waffe_elektronik"
-        (path "/01404002-de85-4f35-b413-98d5163e0060"
+        (path "/9749138d-5476-4991-b12a-e9f07c79da08"
           (reference "#PWR86") (unit 1)
         )

Commit message: Fertigung: JLCPCB-BOM/CPL mit allen Steckern und Tastern (Variante komplett)
- Handlötteile tragen im Schaltplan das Feld "LCSC Hand" statt "LCSC", build_board.py übernimmt es
- jlc_fab.py schreibt zusätzlich *_komplett und *_komplett_externe_antenne (79 Teile, 20 Extended),
  --check prüft den Bedarf der Komplett-Variante; Rotationskorrektur 180° für JST-SH (ungeprüft)
- Schaltplan und Platine neu erzeugt (Geometrie unverändert), Gerber neu, Doku angepasst

Co-Authored-By: Claude Opus 5.5 <noreply@anthropic.com>
Claude-Session: https://claude.ai/code/session_01KkZzubjLKyW9odUwvmxTog
Parts:
- SP1: LCSC Hand (none) -> C225233
Changed lines of the file:
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@@
     (instances
       (project "waffe_elektronik"
-        (path "/9749138d-5476-4991-b12a-e9f07c79da08"
+        (path "/f925400b-2429-4508-9ddf-322832ca444a"
           (reference "U6") (unit 1)
         )
@@
     (instances
       (project "waffe_elektronik"
-        (path "/9749138d-5476-4991-b12a-e9f07c79da08"
+        (path "/f925400b-2429-4508-9ddf-322832ca444a"
           (reference "#PWR70") (unit 1)
         )
@@
     (instances
       (project "waffe_elektronik"
-        (path "/9749138d-5476-4991-b12a-e9f07c79da08"
+        (path "/f925400b-2429-4508-9ddf-322832ca444a"
           (reference "C22") (unit 1)
         )
@@
     (instances
       (project "waffe_elektronik"
-        (path "/9749138d-5476-4991-b12a-e9f07c79da08"
+        (path "/f925400b-2429-4508-9ddf-322832ca444a"
           (reference "#PWR71") (unit 1)
         )
@@
     (instances
       (project "waffe_elektronik"
-        (path "/9749138d-5476-4991-b12a-e9f07c79da08"
+        (path "/f925400b-2429-4508-9ddf-322832ca444a"
           (reference "C23") (unit 1)
         )
@@
     (instances
       (project "waffe_elektronik"
-        (path "/9749138d-5476-4991-b12a-e9f07c79da08"
+        (path "/f925400b-2429-4508-9ddf-322832ca444a"
           (reference "#PWR72") (unit 1)
         )
@@
     (instances
       (project "waffe_elektronik"
-        (path "/9749138d-5476-4991-b12a-e9f07c79da08"
+        (path "/f925400b-2429-4508-9ddf-322832ca444a"
           (reference "#PWR73") (unit 1)
         )
@@
     (instances
       (project "waffe_elektronik"
-        (path "/9749138d-5476-4991-b12a-e9f07c79da08"
+        (path "/f925400b-2429-4508-9ddf-322832ca444a"
           (reference "#PWR74") (unit 1)
         )
@@
     (instances
       (project "waffe_elektronik"
-        (path "/9749138d-5476-4991-b12a-e9f07c79da08"
+        (path "/f925400b-2429-4508-9ddf-322832ca444a"
           (reference "#PWR75") (unit 1)
         )
@@
       (effects (font (size 1.27 1.27)) (justify left) hide)
     )
-    (pin "1")
-    (pin "2")
-    (instances
-      (project "waffe_elektronik"
-        (path "/9749138d-5476-4991-b12a-e9f07c79da08"
+    (property "LCSC Hand" "C225233" (at 0 0 0)
+      (effects (font (size 1.27 1.27)) (justify left) hide)
+    )
+    (pin "1")
+    (pin "2")
+    (instances
+      (project "waffe_elektronik"
+        (path "/f925400b-2429-4508-9ddf-322832ca444a"
           (reference "SP1") (unit 1)
         )
@@
     (instances
       (project "waffe_elektronik"
-        (path "/9749138d-5476-4991-b12a-e9f07c79da08"
+        (path "/f925400b-2429-4508-9ddf-322832ca444a"
           (reference "U14") (unit 1)
         )
@@
     (instances
       (project "waffe_elektronik"
-        (path "/9749138d-5476-4991-b12a-e9f07c79da08"
+        (path "/f925400b-2429-4508-9ddf-322832ca444a"
           (reference "#PWR76") (unit 1)
         )
@@
     (instances
       (project "waffe_elektronik"
-        (path "/9749138d-5476-4991-b12a-e9f07c79da08"
+        (path "/f925400b-2429-4508-9ddf-322832ca444a"
           (reference "C25") (unit 1)
         )
@@
     (instances
       (project "waffe_elektronik"
-        (path "/9749138d-5476-4991-b12a-e9f07c79da08"
+        (path "/f925400b-2429-4508-9ddf-322832ca444a"
           (reference "#PWR77") (unit 1)
         )
@@
     (instances
       (project "waffe_elektronik"
-        (path "/9749138d-5476-4991-b12a-e9f07c79da08"
+        (path "/f925400b-2429-4508-9ddf-322832ca444a"
           (reference "#PWR78") (unit 1)
         )
@@
     (instances
       (project "waffe_elektronik"
-        (path "/9749138d-5476-4991-b12a-e9f07c79da08"
+        (path "/f925400b-2429-4508-9ddf-322832ca444a"
           (reference "R27") (unit 1)
         )
@@
     (instances
       (project "waffe_elektronik"
-        (path "/9749138d-5476-4991-b12a-e9f07c79da08"
+        (path "/f925400b-2429-4508-9ddf-322832ca444a"
           (reference "#PWR79") (unit 1)
         )
@@
     (instances
       (project "waffe_elektronik"
-        (path "/9749138d-5476-4991-b12a-e9f07c79da08"
+        (path "/f925400b-2429-4508-9ddf-322832ca444a"
           (reference "#PWR80") (unit 1)
         )
@@
     (instances
       (project "waffe_elektronik"
-        (path "/9749138d-5476-4991-b12a-e9f07c79da08"
+        (path "/f925400b-2429-4508-9ddf-322832ca444a"
           (reference "J7") (unit 1)
         )
@@
     (instances
       (project "waffe_elektronik"
-        (path "/9749138d-5476-4991-b12a-e9f07c79da08"
+        (path "/f925400b-2429-4508-9ddf-322832ca444a"
           (reference "R37") (unit 1)
         )
@@
     (instances
       (project "waffe_elektronik"
-        (path "/9749138d-5476-4991-b12a-e9f07c79da08"
+        (path "/f925400b-2429-4508-9ddf-322832ca444a"
           (reference "#PWR81") (unit 1)
         )
@@
     (instances
       (project "waffe_elektronik"
-        (path "/9749138d-5476-4991-b12a-e9f07c79da08"
+        (path "/f925400b-2429-4508-9ddf-322832ca444a"
           (reference "#PWR82") (unit 1)
         )
@@
     (instances
       (project "waffe_elektronik"
-        (path "/9749138d-5476-4991-b12a-e9f07c79da08"
+        (path "/f925400b-2429-4508-9ddf-322832ca444a"
           (reference "#PWR83") (unit 1)
         )
@@
     (instances
       (project "waffe_elektronik"
-        (path "/9749138d-5476-4991-b12a-e9f07c79da08"
+        (path "/f925400b-2429-4508-9ddf-322832ca444a"
           (reference "#PWR84") (unit 1)
         )
@@
     (instances
       (project "waffe_elektronik"
-        (path "/9749138d-5476-4991-b12a-e9f07c79da08"
+        (path "/f925400b-2429-4508-9ddf-322832ca444a"
           (reference "C26") (unit 1)
         )
@@
     (instances
       (project "waffe_elektronik"
-        (path "/9749138d-5476-4991-b12a-e9f07c79da08"
+        (path "/f925400b-2429-4508-9ddf-322832ca444a"
           (reference "#PWR85") (unit 1)
         )
@@
     (instances
       (project "waffe_elektronik"
-        (path "/9749138d-5476-4991-b12a-e9f07c79da08"
+        (path "/f925400b-2429-4508-9ddf-322832ca444a"
           (reference "#PWR86") (unit 1)
         )

Commit message: Platine: microSD-Slot gedreht, Ein/Aus über den Drehgeber-Taster, R7 12 Ω, 10 µF am Slot
- J7: Karte wird auf der Kontaktseite eingesteckt (Datenblatt TF-018) -> Slot gedreht, Kontakte und
  Öffnung an der Unterkante, SD-Leitungen neu verlegt
- Soft-Power: Q4 (AO3401A) trennt den Akku von BAT_SW, Taster an J5.2 schaltet über D6 (BAT54CW) ein,
  IO21 hält über Q5, IO9 liest den Taster; Lasche oben links 18,6 x 9 mm mit den neuen Teilen,
  Leitungen auf B.Cu über die Oberkante, Akku-Plus über In2
- R7 12 Ω (C17913), C28 10 µF an der microSD-Versorgung
- Gerber, BOM/CPL (alle Varianten), Mouser-BOM, Renders und Doku neu

Co-Authored-By: Claude Opus 5.5 <noreply@anthropic.com>
Claude-Session: https://claude.ai/code/session_01KkZzubjLKyW9odUwvmxTog
Parts:
- added C28: 10u, Capacitor_SMD:C_0603_1608Metric, symbol Device:C
Connections:
- net 3V3_MCU: now also C28.1
- net GND: now also C28.2

Commit message: Platine: Stecker zusammengelegt, Basic-Teile, MOSFET-Pegelwandler, Flash optional, Kabel-3V3 über 10 Ω, breitere 5-V- und Akku-Wege
Co-Authored-By: Claude Opus 5.5 <noreply@anthropic.com>
Claude-Session: https://claude.ai/code/session_01KkZzubjLKyW9odUwvmxTog
Parts:
- C25: LCSC C14663 -> (none); LCSC Option (none) -> C14663
- R27: LCSC C25804 -> (none); LCSC Option (none) -> C25804
- U14: LCSC C2928927 -> (none); LCSC Option (none) -> C2928927
