File: kicad/waffe_elektronik/bedienung_aktoren.kicad_sch (KiCad schematic)
At the start: 24 parts, among them J1 WS2812 HP-Streifen, J4 OLED I²C (Qwiic), J5 Drehgeber, M1 Vibromotor, Q1 AO3400A, Q2 AO3400A, SW1 Taster, SW2 Taster, U5 74HCT125

Commit message: Platine: günstigere JLC-Teile, Option ESP32-S3-WROOM-1U mit externer Antenne
- Flash ZD35Q1GC-IB, Kondensatoren/Dioden/Widerstände auf Basic-Teile und 0402, Layout angepasst
- WROOM-1U auf demselben Footprint: eigene JLCPCB-BOM/CPL (Modulmitte 3,15 mm versetzt),
  Mouser-Option mit Pigtail RP-SMA/U.FL und Knick-Stabantenne, 3D-Modell des 1U
- Gerber, BOM, CPL, Renders und Bestelllisten neu erzeugt

Co-Authored-By: Claude Opus 5.5 <noreply@anthropic.com>
Claude-Session: https://claude.ai/code/session_01KkZzubjLKyW9odUwvmxTog
Parts:
- C10: LCSC C723734 -> C23742
- C7: LCSC C49066 -> C23742
- D1: value SS14 -> B5819W; footprint Diode_SMD:D_SOD-123F -> Diode_SMD:D_SOD-123; LCSC C2909920 -> C8598
- J1: LCSC C225234 -> (none)
- J4, J5: LCSC C160404 -> (none)
- LED1, M1, SW1, SW2: LCSC C160402 -> (none)

Commit message: Fertigung: JLCPCB-BOM/CPL mit allen Steckern und Tastern (Variante komplett)
- Handlötteile tragen im Schaltplan das Feld "LCSC Hand" statt "LCSC", build_board.py übernimmt es
- jlc_fab.py schreibt zusätzlich *_komplett und *_komplett_externe_antenne (79 Teile, 20 Extended),
  --check prüft den Bedarf der Komplett-Variante; Rotationskorrektur 180° für JST-SH (ungeprüft)
- Schaltplan und Platine neu erzeugt (Geometrie unverändert), Gerber neu, Doku angepasst

Co-Authored-By: Claude Opus 5.5 <noreply@anthropic.com>
Claude-Session: https://claude.ai/code/session_01KkZzubjLKyW9odUwvmxTog
Parts:
- J1: LCSC Hand (none) -> C225234
- J4, J5: LCSC Hand (none) -> C160404
- LED1, M1, SW1, SW2: LCSC Hand (none) -> C160402

Commit message: Platine: microSD-Slot gedreht, Ein/Aus über den Drehgeber-Taster, R7 12 Ω, 10 µF am Slot
- J7: Karte wird auf der Kontaktseite eingesteckt (Datenblatt TF-018) -> Slot gedreht, Kontakte und
  Öffnung an der Unterkante, SD-Leitungen neu verlegt
- Soft-Power: Q4 (AO3401A) trennt den Akku von BAT_SW, Taster an J5.2 schaltet über D6 (BAT54CW) ein,
  IO21 hält über Q5, IO9 liest den Taster; Lasche oben links 18,6 x 9 mm mit den neuen Teilen,
  Leitungen auf B.Cu über die Oberkante, Akku-Plus über In2
- R7 12 Ω (C17913), C28 10 µF an der microSD-Versorgung
- Gerber, BOM/CPL (alle Varianten), Mouser-BOM, Renders und Doku neu

Co-Authored-By: Claude Opus 5.5 <noreply@anthropic.com>
Claude-Session: https://claude.ai/code/session_01KkZzubjLKyW9odUwvmxTog
Parts:
- R7: value 10 -> 12; LCSC C17903 -> C17913
Connections:
- net BAT_P renamed BAT_SW
- net ENC_SW renamed PWR_KEY

Commit message: Platine: IP5306 (2 A Laden + 5 V) statt MT3608/MCP73831, Ein/Aus über KEY, eigener I²C-Bus
Co-Authored-By: Claude Opus 5.5 <noreply@anthropic.com>
Claude-Session: https://claude.ai/code/session_01KkZzubjLKyW9odUwvmxTog
Connections:
- net BAT_SW renamed BAT_P

Commit message: Platine: Stecker zusammengelegt, Basic-Teile, MOSFET-Pegelwandler, Flash optional, Kabel-3V3 über 10 Ω, breitere 5-V- und Akku-Wege
Co-Authored-By: Claude Opus 5.5 <noreply@anthropic.com>
Claude-Session: https://claude.ai/code/session_01KkZzubjLKyW9odUwvmxTog
Parts:
- removed C21: 100n, Capacitor_SMD:C_0603_1608Metric, symbol Device:C
- removed U5: 74HCT125, Package_SO:TSSOP-14_4.4x5mm_P0.65mm, symbol lasertag:74AHCT125
- added C32: 22u, Capacitor_SMD:C_0805_2012Metric, symbol Device:C
- added J8: Abzug + Nachladen, Connector_JST:JST_SH_SM03B-SRSS-TB_1x03-1MP_P1.00mm_Horizontal, symbol Connector_Generic:Conn_01x03
- added Q4: 2N7002, Package_TO_SOT_SMD:SOT-23, symbol Transistor_FET:2N7002
- added R25: 1k, Resistor_SMD:R_0603_1608Metric, symbol Device:R
- added R8: 22, Resistor_SMD:R_1206_3216Metric, symbol Device:R
- C10, C7: value 100u -> 22u; footprint Capacitor_SMD:C_1210_3225Metric -> Capacitor_SMD:C_0805_2012Metric; LCSC C23742 -> C45783
- LED1, SW1, SW2: footprint Connector_JST:JST_SH_SM02B-SRSS-TB_1x02-1MP_P1.00mm_Horizontal -> (none); LCSC Hand C160402 -> (none)
- R7: value 12 -> 22; LCSC C17913 -> C17958
Connections:
- net 3V3_MCU: now also Q4.1 (G)
- net 5V_PERIPH: now also C32.1, R25.1
- net BAT_P: now also R8.1
- net GND: now also C32.2, J8.2 (Pin_2)
- net RELOAD: now also J8.3 (Pin_3)
- net TRIGGER: now also J8.1 (Pin_1)
- net WS2812_DIN_3V3: now also Q4.2 (S)
- net IR_LED_K: now reaches LED1.1 (K), Q1.3 (D)
- net IR_LED_A: now reaches LED1.2 (A), R7.2
- net IR_LED_A: now also R8.2
- net at R15.1: now also Q4.3 (D), R25.2
- no-connect marks 3 -> 0
Other:
- note added: "LED an der Waffe (J6)"
- note added: "WS2812 (5 V) über Pegelwandler (MOSFET)"
- note removed: "WS2812 (5 V) über Pegelwandler"
- note removed: "unbenutzte Gatter: Eingänge + /OE auf GND"
