File: kicad/waffe_elektronik/sensoren.kicad_sch (KiCad schematic)
At the start: 25 parts, among them J2 GX16 7-polig, J6 TSOP 6 (Waffe), U10 TSOP34838, U11 TSOP34838, U13 TSOP34838, U7 TSOP34838, U8 TSOP34838, U9 TSOP34838

Commit message: Platine: günstigere JLC-Teile, Option ESP32-S3-WROOM-1U mit externer Antenne
- Flash ZD35Q1GC-IB, Kondensatoren/Dioden/Widerstände auf Basic-Teile und 0402, Layout angepasst
- WROOM-1U auf demselben Footprint: eigene JLCPCB-BOM/CPL (Modulmitte 3,15 mm versetzt),
  Mouser-Option mit Pigtail RP-SMA/U.FL und Knick-Stabantenne, 3D-Modell des 1U
- Gerber, BOM, CPL, Renders und Bestelllisten neu erzeugt

Co-Authored-By: Claude Opus 5.5 <noreply@anthropic.com>
Claude-Session: https://claude.ai/code/session_01KkZzubjLKyW9odUwvmxTog
Parts:
- J2: LCSC C160406 -> (none)
- J6: LCSC C7430445 -> (none)

Commit message: Fertigung: JLCPCB-BOM/CPL mit allen Steckern und Tastern (Variante komplett)
- Handlötteile tragen im Schaltplan das Feld "LCSC Hand" statt "LCSC", build_board.py übernimmt es
- jlc_fab.py schreibt zusätzlich *_komplett und *_komplett_externe_antenne (79 Teile, 20 Extended),
  --check prüft den Bedarf der Komplett-Variante; Rotationskorrektur 180° für JST-SH (ungeprüft)
- Schaltplan und Platine neu erzeugt (Geometrie unverändert), Gerber neu, Doku angepasst

Co-Authored-By: Claude Opus 5.5 <noreply@anthropic.com>
Claude-Session: https://claude.ai/code/session_01KkZzubjLKyW9odUwvmxTog
Parts:
- J2: LCSC Hand (none) -> C160406
- J6: LCSC Hand (none) -> C7430445

Commit message: Platine: Stecker zusammengelegt, Basic-Teile, MOSFET-Pegelwandler, Flash optional, Kabel-3V3 über 10 Ω, breitere 5-V- und Akku-Wege
Co-Authored-By: Claude Opus 5.5 <noreply@anthropic.com>
Claude-Session: https://claude.ai/code/session_01KkZzubjLKyW9odUwvmxTog
Parts:
- removed J6: TSOP 6 (Waffe), Connector_JST:JST_SH_SM03B-SRSS-TB_1x03-1MP_P1.00mm_Horizontal, symbol Connector_Generic:Conn_01x03
- added J6: IR-LED + TSOP 6, Connector_JST:JST_SH_SM05B-SRSS-TB_1x05-1MP_P1.00mm_Horizontal, symbol Connector_Generic:Conn_01x05
- added R35: 10, Resistor_SMD:R_0402_1005Metric, symbol Device:R
- added R36: 10, Resistor_SMD:R_0603_1608Metric, symbol Device:R
Connections:
- net 3V3_MCU: now also R35.1, R36.1; no longer J2.1 (Pin_1), R16.1, R17.1, R18.1, R19.1, R20.1, R26.1
- net GND: now also J6.3 (Pin_3)
- net TSOP6_OUT: now also J6.5 (Pin_5)
- new net 3V3_J6: J6.4 (Pin_4), R26.1, R36.2
- new net 3V3_WESTE: J2.1 (Pin_1), R16.1, R17.1, R18.1, R19.1, R20.1, R35.2
- new net IR_LED_A: J6.1 (Pin_1)
- new net IR_LED_K: J6.2 (Pin_2)
Other:
- note added: "IR-LED + TSOP 6 (an der Waffe, Stecker J6)"
- note added: "Kabel zu IR-LED und Sensor vorn an der Waffe"
- note removed: "Kabel zum Sensor an der Waffe"
- note removed: "TSOP 6 (an der Waffe, jenseits des Steckers)"

Commit message: Platine: Herstellerzeichen mit Borg-Würfel unter U2, Schaltplan: Westen-TSOP-Ausgänge auf Steckerseite
Co-Authored-By: Claude Opus 5.5 <noreply@anthropic.com>
Claude-Session: https://claude.ai/code/session_01KkZzubjLKyW9odUwvmxTog
Connections:
- net TSOP1_J: now also U7.1 (OUT)
- net TSOP1_OUT: no longer U7.1 (OUT)
- net TSOP2_J: now also U8.1 (OUT)
- net TSOP2_OUT: no longer U8.1 (OUT)
- net TSOP3_J: now also U9.1 (OUT)
- net TSOP3_OUT: no longer U9.1 (OUT)
- net TSOP4_J: now also U10.1 (OUT)
- net TSOP4_OUT: no longer U10.1 (OUT)
- net TSOP5_J: now also U11.1 (OUT)
- net TSOP5_OUT: no longer U11.1 (OUT)
