File: kicad/waffe_elektronik/waffe_elektronik.kicad_pcb (KiCad board)
At the start: 4 copper layers, 59.6 x 55 mm, 89 parts, among them J1 WS2812 HP-Streifen, J2 GX16 7-polig, J3 USB-C (Flashen + Laden), J4 OLED I²C (Qwiic), J5 Drehgeber, J6 IR-LED + TSOP 6, J7 TF-018, J8 Abzug + Nachladen, M1 Vibromotor, Q1 AO3400A, Q2 AO3400A, Q3 FS8205A, Q4 2N7002, SW3 RESET, SW4 BOOT, U1 IP5306-I2C, U12 USBLC6-2SC6, U14 ZD35Q1GC-IB, U15 DW01A, U16 TPS22810, U2 AMS1117-3.3, U4 ESP32-S3-WROOM-1-N16R8, U6 MAX98357A

Commit message: Platine: nur Logo + URL unter U2, weißer Lötstopplack mit schwarzem Druck (Stackup, Renders)
Co-Authored-By: Claude Opus 5.5 <noreply@anthropic.com>
Claude-Session: https://claude.ai/code/session_01KkZzubjLKyW9odUwvmxTog
Other:
- board text removed: "made by"

Commit message: Platine: Herstellertexte in Orbitron / Share Tech Mono als Silk-Polygone (Schriften in fonts/)
Co-Authored-By: Claude Opus 5.5 <noreply@anthropic.com>
Claude-Session: https://claude.ai/code/session_01KkZzubjLKyW9odUwvmxTog
Routing:
- net GND: vias 144 -> 140
Other:
- board text removed: "github.com/G5K-org/open-lasertag"
- board text removed: "lucas.giesecke.cc"
- board text removed: "open-lasertag v1"
